Commit message: Phase 3 complete: CNN line follower tracks curves with recovery behavior

File: src/line_follower/urdf/robot.urdf.xacro (robot description, xacro)
@@ -80,5 +80,5 @@
       <origin xyz="0 ${y_reflect * wheel_separation/2} 0"
               rpy="${pi/2} 0 0"/>
-      <axis xyz="0 0 1"/>
+      <axis xyz="0 0 -1"/>
     </joint>
 </xacro:macro>
@@ -176,3 +176,14 @@
     </sensor>
 </gazebo>
+<gazebo>
+    <plugin name="diff_drive" filename="libgazebo_ros_diff_drive.so">
+      <left_joint>left_wheel_joint</left_joint>
+      <right_joint>right_wheel_joint</right_joint>
+      <wheel_separation>0.22</wheel_separation>
+      <wheel_diameter>0.10</wheel_diameter>
+      <command_topic>cmd_vel</command_topic>
+      <publish_odom>true</publish_odom>
+      <robot_base_frame>base_link</robot_base_frame>
+    </plugin>
+  </gazebo>
 </robot>
